Commit message: fix: frame orientations

File: data/bhl_arm/urdf/bhl_arm.urdf (robot description, URDF)
Before this commit: robot bhl_arm, 17 links, 16 joints
Links:
- link base: mass 1.10336 -> 1.35672
- link left_fingertip: geometry collision cylinder length=0.07 radius=0.008; visual mesh filename=../meshes/left_fingertip_visual.stl
- link left_wrist_yaw: mass 0.522 -> 0.6
- link right_fingertip: geometry collision cylinder length=0.07 radius=0.008; visual mesh filename=../meshes/right_fingertip_visual.stl
- link right_wrist_yaw: mass 0.522 -> 0.6
Joints:
- joint left_dummy_fingertip: origin xyz=-0.215 -0.007 -0.0005 rpy=-1.5708 0 1.5708 -> xyz=-0.007 0.215 -0.0005 rpy=-1.5708 0 0
- joint left_elbow_pitch: limit lower=-2.35619 upper=0 effort=100 velocity=100 -> lower=-0 upper=2.35619 effort=100 velocity=100; origin xyz=0.01 0.0286 -0.08 rpy=-1.5708 -1.5708 0 -> xyz=0.01 0.0286 -0.08 rpy=-1.5708 0 -0
- joint left_shoulder_pitch: limit lower=-3.14159 upper=0.785398 effort=100 velocity=100 -> lower=-0.785398 upper=3.14159 effort=100 velocity=100; origin xyz=-0 0.0506077 0.383054 rpy=-1.39626 0 -0 -> xyz=0 0.0506077 0.683054 rpy=-1.39626 0 -0
- joint left_shoulder_roll: limit lower=-0.174533 upper=3.31613 effort=100 velocity=100 -> lower=-3.31613 upper=0.174533 effort=100 velocity=100; origin xyz=0.0286 0 0.04 rpy=-1.5708 0 -1.5708 -> xyz=0.0286 0 0.04 rpy=1.5708 0.174533 1.5708
- joint left_shoulder_yaw: origin xyz=-0.12 -0 -0.0286 rpy=3.14159 -1.5708 0 -> xyz=0 0.12 -0.0286 rpy=1.5708 -1.5708 0
- joint left_wrist_pitch: origin xyz=0 0.025 -0.025 rpy=-1.5708 0 -0 -> xyz=0.025 0 -0.025 rpy=0 1.5708 0
- joint left_wrist_roll: origin xyz=-0.0250003 3.4253e-08 -0.14 rpy=0 -1.5708 0 -> xyz=3.4253e-08 0.0250003 -0.14 rpy=-1.5708 -0 -0
- joint left_wrist_yaw: origin xyz=-0.06 -0.00999972 -0.0286 rpy=-0 1.5708 0 -> xyz=-0.00999972 0.06 -0.0286 rpy=1.5708 -0 -0
- joint right_dummy_fingertip: origin xyz=0.215 -0.007 -0.0005 rpy=1.5708 0 1.5708 -> xyz=0.007 0.215 -0.0005 rpy=1.5708 -0 -3.14159
- joint right_elbow_pitch: origin xyz=0.01 -0.0286 -0.08 rpy=-1.5708 1.5708 0 -> xyz=0.01 -0.0286 -0.08 rpy=-1.5708 0 -0
- joint right_shoulder_pitch: origin xyz=-0 -0.0506077 0.383054 rpy=-1.74533 -0 -0 -> xyz=-0 -0.0506077 0.683054 rpy=-1.74533 0 -0
- joint right_shoulder_roll: limit lower=-3.31613 upper=0.174533 effort=100 velocity=100 -> lower=-0.174533 upper=3.31613 effort=100 velocity=100; origin xyz=0.0286 0 -0.04 rpy=1.5708 0 1.5708 -> xyz=0.0286 -0 -0.04 rpy=-1.5708 0.174533 -1.5708
- joint right_shoulder_yaw: origin xyz=0.12 0 -0.0286 rpy=0 -1.5708 0 -> xyz=-0 0.12 -0.0286 rpy=1.5708 -1.5708 0
- joint right_wrist_pitch: origin xyz=-0 0.025 0.025 rpy=1.5708 0 -3.14159 -> xyz=0.025 0 0.025 rpy=0 1.5708 0
- joint right_wrist_roll: origin xyz=-0.0250003 1.9152e-08 -0.14 rpy=3.14159 -1.5708 0 -> xyz=-1.9152e-08 -0.0250003 -0.14 rpy=-1.5708 0 -0
- joint right_wrist_yaw: origin xyz=0.0598068 0.0100599 0.0286 rpy=0 -1.5708 0 -> xyz=-0.00999973 0.06 0.0286 rpy=1.5708 -0 -0

Commit message: fix: joint limits

File: data/bhl_arm/urdf/bhl_arm.urdf (robot description, URDF)
Before this commit: robot bhl_arm, 17 links, 16 joints
Joints:
- joint left_dummy_fingertip: origin xyz=-0.007 0.215 -0.0005 rpy=-1.5708 0 0 -> xyz=-0.007 0.215 -0.0005 rpy=-1.5708 0 -0
- joint left_elbow_pitch: limit lower=-0 upper=2.35619 effort=100 velocity=100 -> lower=-2.35619 upper=0 effort=100 velocity=100
- joint left_shoulder_pitch: limit lower=-0.785398 upper=3.14159 effort=100 velocity=100 -> lower=-3.14159 upper=0.785398 effort=100 velocity=100
- joint left_shoulder_roll: limit lower=-3.31613 upper=0.174533 effort=100 velocity=100 -> lower=-1.5708 upper=1.91986 effort=100 velocity=100
- joint left_shoulder_yaw: origin xyz=0 0.12 -0.0286 rpy=1.5708 -1.5708 0 -> xyz=-0 0.12 -0.0286 rpy=1.5708 -1.5708 0
- joint left_wrist_pitch: origin xyz=0.025 0 -0.025 rpy=0 1.5708 0 -> xyz=0.025 0 -0.025 rpy=-0 1.5708 0
- joint left_wrist_yaw: origin xyz=-0.00999972 0.06 -0.0286 rpy=1.5708 -0 -0 -> xyz=-0.00999972 0.06 -0.0286 rpy=1.5708 0 0
- joint right_dummy_fingertip: origin xyz=0.007 0.215 -0.0005 rpy=1.5708 -0 -3.14159 -> xyz=0.007 0.215 -0.0005 rpy=1.5708 0 3.14159
- joint right_elbow_pitch: origin xyz=0.01 -0.0286 -0.08 rpy=-1.5708 0 -0 -> xyz=0.01 -0.0286 -0.08 rpy=-1.5708 -0 0
- joint right_shoulder_pitch: origin xyz=-0 -0.0506077 0.683054 rpy=-1.74533 0 -0 -> xyz=-0 -0.0506077 0.683054 rpy=-1.74533 -0 0
- joint right_shoulder_roll: limit lower=-0.174533 upper=3.31613 effort=100 velocity=100 -> lower=-1.91986 upper=1.5708 effort=100 velocity=100; origin xyz=0.0286 -0 -0.04 rpy=-1.5708 0.174533 -1.5708 -> xyz=0.0286 0 -0.04 rpy=-1.5708 0.174533 -1.5708
- joint right_shoulder_yaw: origin xyz=-0 0.12 -0.0286 rpy=1.5708 -1.5708 0 -> xyz=0 0.12 -0.0286 rpy=1.5708 -1.5708 0
- joint right_wrist_yaw: origin xyz=-0.00999973 0.06 0.0286 rpy=1.5708 -0 -0 -> xyz=-0.00999973 0.06 0.0286 rpy=1.5708 0 -0
